Commit message: docs: README 업데이트 및 기타 파일 수정

File: urdf/mid360.xacro (robot description, xacro)
@@ -12,4 +12,5 @@
   <xacro:property name="width" value="0.06" />
   <xacro:property name="height" value="0.06" />
+<xacro:property name="livox_share" value="$(find ros2_livox_simulation)"/>
   <xacro:macro name="box_inertia" params="m w h d">
     <inertial>
@@ -24,5 +25,5 @@
   <visual>
         <geometry>
-            <box size="${length} ${width} ${height}"/>
+            <mesh filename="file://${livox_share}/meshes/mid-360-scaled.dae"/>
         </geometry>
   </visual>

Commit message: modified mass

File: urdf/mid360.xacro (robot description, xacro)
@@ -8,5 +8,5 @@
   <xacro:property name="noise_mean" value="0.0"/>
   <xacro:property name="noise_stddev" value="0.01"/>
-  <xacro:property name="mass" value="0.4" />
+  <xacro:property name="mass" value="0.0001" />
   <xacro:property name="length" value="0.1" />
   <xacro:property name="width" value="0.06" />

Commit message: Bug: min_range should be zero

File: urdf/mid360.xacro (robot description, xacro)
@@ -2,5 +2,5 @@
 <robot xmlns:xacro="http://ros.org/wiki/xacro">
   <xacro:property name="M_PI" value="3.1415926"/>
-  <xacro:property name="laser_min_range" value="0.1"/>
+  <xacro:property name="laser_min_range" value="0.0"/>
   <xacro:property name="laser_max_range" value="200.0"/>
   <xacro:property name="samples" value="40000"/>
